File: atari-joystick-slim/layouts/default/default.kicad_pcb (KiCad board)
At the start: 4 copper layers, 30 x 16 mm, 19 parts

Commit message: フルカラー LED を WS2812B-2020-V6 (C52917434) に置き換え
x68000-keyboard / atari-joystick-slim / wireless-combo のステータス LED を
旧品 WS2812B-2020 (C965555, 電源 3.5V〜) から同外形・同ピン配置の
WS2812B-2020-V6 (電源 3.3〜5.3V) に置き換え、3.3V 給電を定格内にする。

- parts/Worldsemi_WS2812B_2020_V6 を追加 (3D モデルは旧品のものを流用)、旧部品を削除
- パッド位置はほぼ同一のため配線は不変、ゾーンのみ再充填 (DRC 0/0)
- x68000-keyboard v1.0.1 / combo v1.0.0 の製造データを再生成
- atari-joystick (rev 1.0.0 製造済み) は変更しない

Co-Authored-By: Claude Opus 5.5 <noreply@anthropic.com>
Parts:
- LED2: footprint Worldsemi_WS2812B_2020:LED-SMD_4P-L2.0-W2.0-TL_WS2812B-2020 -> Worldsemi_WS2812B_2020_V6:LED-SMD_4P-L2.2-W2.0-P1.00_WS2815C-2020-4P
