File: x68000-keyboard/layouts/default/default.kicad_pcb (KiCad board)
At the start: 4 copper layers, 29.6 x 12.2 mm, 19 parts

Commit message: フルカラー LED を WS2812B-2020-V6 (C52917434) に置き換え
x68000-keyboard / atari-joystick-slim / wireless-combo のステータス LED を
旧品 WS2812B-2020 (C965555, 電源 3.5V〜) から同外形・同ピン配置の
WS2812B-2020-V6 (電源 3.3〜5.3V) に置き換え、3.3V 給電を定格内にする。

- parts/Worldsemi_WS2812B_2020_V6 を追加 (3D モデルは旧品のものを流用)、旧部品を削除
- パッド位置はほぼ同一のため配線は不変、ゾーンのみ再充填 (DRC 0/0)
- x68000-keyboard v1.0.1 / combo v1.0.0 の製造データを再生成
- atari-joystick (rev 1.0.0 製造済み) は変更しない

Co-Authored-By: Claude Opus 5.5 <noreply@anthropic.com>
Parts:
- LED2: footprint Worldsemi_WS2812B_2020:LED-SMD_4P-L2.0-W2.0-TL_WS2812B-2020 -> Worldsemi_WS2812B_2020_V6:LED-SMD_4P-L2.2-W2.0-P1.00_WS2815C-2020-4P
Changed lines of the file:
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@@
 		)
 	)
-	(footprint "Worldsemi_WS2812B_2020:LED-SMD_4P-L2.0-W2.0-TL_WS2812B-2020"
+	(footprint "Worldsemi_WS2812B_2020_V6:LED-SMD_4P-L2.2-W2.0-P1.00_WS2815C-2020-4P"
 		(layer "F.Cu")
 		(at 162.2 100.8)
@@
 			)
 		)
-		(property "Datasheet" "https://www.lcsc.com/datasheet/lcsc_datasheet_2012110135_Worldsemi-WS2812B-2020_C965555.pdf"
+		(property "Datasheet" "https://www.lcsc.com/datasheet/C52917434.pdf"
 			(at 0 0 0)
 			(layer "User.9")
@@
 			)
 		)
-		(property "LCSC" "C965555"
+		(property "LCSC" "C52917434"
 			(at 0 0 0)
 			(layer "User.9")
@@
 			)
 		)
-		(property "Partnumber" "WS2812B-2020"
+		(property "Partnumber" "WS2812B-2020-V6"
 			(at 0 0 0)
 			(layer "User.9")
@@
 			)
 		)
-		(property "lcsc_id" "C965555"
+		(property "lcsc_id" "C52917434"
 			(at 0 0 0)
 			(layer "User.9")
@@
 			)
 		)
-		(attr smd)
+		(attr through_hole)
 		(fp_line
-			(start -1.3 -1.15)
-			(end -1.3 -1.14)
-			(stroke
-				(width 0.25)
-				(type solid)
-			)
-			(layer "F.SilkS")
-		)
-		(fp_line
-			(start -1 1.1)
-			(end 1 1.1)
+			(start -0.4 1.13)
+			(end -1 1.13)
 			(stroke
 				(width 0.15)
@@
 		)
 		(fp_line
-			(start -0.25 -0.75)
-			(end -0.25 0.7)
+			(start -0.4 1.13)
+			(end 0.33 1.13)
 			(stroke
 				(width 0.15)
@@
 		)
 		(fp_line
-			(start -0.25 -0.75)
-			(end -0.1 -0.75)
+			(start -0.34 -1.13)
+			(end -1 -1.13)
 			(stroke
 				(width 0.15)
@@
 		)
 		(fp_line
-			(start -0.1 -0.75)
-			(end -0.1 0.65)
+			(start -0.2 0.8)
+			(end -0.2 -0.8)
 			(stroke
-				(width 0.15)
+				(width 0.4)
 				(type solid)
 			)
@@
 		)
 		(fp_line
-			(start -0.1 0.65)
-			(end -0.1 0.7)
+			(start 0.33 1.13)
+			(end 1 1.13)
 			(stroke
 				(width 0.15)
@@
 		)
 		(fp_line
-			(start -0.1 0.7)
-			(end -0.25 0.7)
+			(start 0.4 -1.13)
+			(end -0.34 -1.13)
 			(stroke
 				(width 0.15)
@@
 		)
 		(fp_line
-			(start 1 -1.1)
-			(end -1 -1.1)
+			(start 0.4 -1.13)
+			(end 1 -1.13)
 			(stroke
 				(width 0.15)
@@
 		)
 		(pad "1" smd rect
-			(at -0.92 -0.55)
-			(size 0.9 0.7)
+			(at -0.87 -0.55 180)
+			(size 0.8 0.8)
 			(layers "F.Cu" "F.Mask" "F.Paste")
 			(net 44 "dout")
 		)
 		(pad "2" smd rect
-			(at -0.92 0.55)
-			(size 0.9 0.7)
+			(at -0.87 0.55 180)
+			(size 0.8 0.8)
 			(layers "F.Cu" "F.Mask" "F.Paste")
 			(net 11 "GND")
 		)
 		(pad "3" smd rect
-			(at 0.92 0.55)
-			(size 0.9 0.7)
+			(at 0.86 0.55 180)
+			(size 0.8 0.8)
 			(layers "F.Cu" "F.Mask" "F.Paste")
 			(net 45 "din")
 		)
 		(pad "4" smd rect
-			(at 0.92 -0.55)
-			(size 0.9 0.7)
+			(at 0.86 -0.55 180)
+			(size 0.8 0.8)
 			(layers "F.Cu" "F.Mask" "F.Paste")
 			(net 41 "VDD33")
 		)
 		(embedded_fonts no)
-		(model "${KIPRJMOD}/../../parts/Worldsemi_WS2812B_2020/LED-SMD_4P-L2.0-W2.0-H0.8-TL_WS2812B-2020.step"
+		(model "${KIPRJMOD}/../../parts/Worldsemi_WS2812B_2020_V6/WS2812B-2020-V6.step"
 			(offset
 				(xyz 0 0 -0)
@@
 		(property "Reference" "R5"
 			(at -1.4 0 0)
-			(unlocked yes)
 			(layer "F.SilkS")
 			(effects
@@
 			)
 		)
-		(property "Datasheet" "https://www.lcsc.com/datasheet/lcsc_datasheet_2205311900_UNI-ROYAL-Uniroyal-Elec-0402WGF4700TCE_C25117.pdf"
+		(property "Datasheet" ""
 			(at 0 0 90)
 			(layer "User.9")
@@
 			)
 		)
-		(property "Manufacturer" "UNI-ROYAL(Uniroyal Elec)"
+		(property "Manufacturer" "UNI-ROYAL"
 			(at 0 0 90)
 			(layer "User.9")
@@
 			)
 		)
-		(property "Datasheet" "https://www.lcsc.com/datasheet/lcsc_datasheet_2304140030_Samsung-Electro-Mechanics-CL05A105KA5NQNC_C52923.pdf"
+		(property "Datasheet" ""
 			(at 0 0 0)
 			(layer "User.9")
@@
 			)
 		)
-		(property "PARAM_capacitance" "{\"type\": \"Quantity_Interval_Disjoint\", \"data\": {\"intervals\": {\"type\": \"Numeric_Interval_Disjoint\", \"data\": {\"intervals\": [{\"type\": \"Numeric_Interval\", \"data\": {\"min\": 8.999999985098838e-07, \"max\": 1.100000001490116e-06}}]}}, \"unit\": \"farad\"}}"
+		(property "PARAM_capacitance" "{\"type\": \"Quantity_Interval_Disjoint\", \"data\": {\"intervals\": {\"type\": \"Numeric_Interval_Disjoint\", \"data\": {\"intervals\": [{\"type\": \"Numeric_Interval\", \"data\": {\"min\": 9e-07, \"max\": 1.1e-06}}]}}, \"unit\": \"farad\"}}"
 			(at 0 0 0)
 			(layer "User.9")
@@
 			)
 		)
-		(property "Datasheet" "https://www.lcsc.com/datasheet/lcsc_datasheet_2304140030_Samsung-Electro-Mechanics-CL05A105KA5NQNC_C52923.pdf"
+		(property "Datasheet" ""
 			(at 0 0 0)
 			(layer "User.9")
@@
 			)
 		)
-		(property "PARAM_capacitance" "{\"type\": \"Quantity_Interval_Disjoint\", \"data\": {\"intervals\": {\"type\": \"Numeric_Interval_Disjoint\", \"data\": {\"intervals\": [{\"type\": \"Numeric_Interval\", \"data\": {\"min\": 8.999999985098838e-07, \"max\": 1.100000001490116e-06}}]}}, \"unit\": \"farad\"}}"
+		(property "PARAM_capacitance" "{\"type\": \"Quantity_Interval_Disjoint\", \"data\": {\"intervals\": {\"type\": \"Numeric_Interval_Disjoint\", \"data\": {\"intervals\": [{\"type\": \"Numeric_Interval\", \"data\": {\"min\": 9e-07, \"max\": 1.1e-06}}]}}, \"unit\": \"farad\"}}"
 			(at 0 0 0)
 			(layer "User.9")
@@
 			)
 		)
-		(property "Datasheet" "https://www.lcsc.com/datasheet/lcsc_datasheet_2304140030_Samsung-Electro-Mechanics-CL05B104KO5NNNC_C1525.pdf"
+		(property "Datasheet" ""
 			(at 0 0 0)
 			(layer "User.9")
@@
 			)
 		)
-		(property "PARAM_capacitance" "{\"type\": \"Quantity_Interval_Disjoint\", \"data\": {\"intervals\": {\"type\": \"Numeric_Interval_Disjoint\", \"data\": {\"intervals\": [{\"type\": \"Numeric_Interval\", \"data\": {\"min\": 8.99999998509884e-08, \"max\": 1.1000000014901162e-07}}]}}, \"unit\": \"farad\"}}"
+		(property "PARAM_capacitance" "{\"type\": \"Quantity_Interval_Disjoint\", \"data\": {\"intervals\": {\"type\": \"Numeric_Interval_Disjoint\", \"data\": {\"intervals\": [{\"type\": \"Numeric_Interval\", \"data\": {\"min\": 9.000000000000001e-08, \"max\": 1.1000000000000002e-07}}]}}, \"unit\": \"farad\"}}"
 			(at 0 0 0)
 			(layer "User.9")
@@
 			)
 		)
-		(property "Datasheet" "https://www.lcsc.com/datasheet/lcsc_datasheet_2206010045_UNI-ROYAL-Uniroyal-Elec-0402WGF5101TCE_C25905.pdf"
+		(property "Datasheet" ""
 			(at 0 0 0)
 			(layer "User.9")
@@
 			)
 		)
-		(property "Manufacturer" "UNI-ROYAL(Uniroyal Elec)"
+		(property "Manufacturer" "UNI-ROYAL"
 			(at 0 0 0)
 			(layer "User.9")
@@
 			)
 		)
-		(property "Datasheet" "https://www.lcsc.com/datasheet/lcsc_datasheet_2304140030_Samsung-Electro-Mechanics-CL05B104KO5NNNC_C1525.pdf"
+		(property "Datasheet" ""
 			(at 0 0 0)
 			(layer "User.9")
@@
 			)
 		)
-		(property "PARAM_capacitance" "{\"type\": \"Quantity_Interval_Disjoint\", \"data\": {\"intervals\": {\"type\": \"Numeric_Interval_Disjoint\", \"data\": {\"intervals\": [{\"type\": \"Numeric_Interval\", \"data\": {\"min\": 8.99999998509884e-08, \"max\": 1.1000000014901162e-07}}]}}, \"unit\": \"farad\"}}"
+		(property "PARAM_capacitance" "{\"type\": \"Quantity_Interval_Disjoint\", \"data\": {\"intervals\": {\"type\": \"Numeric_Interval_Disjoint\", \"data\": {\"intervals\": [{\"type\": \"Numeric_Interval\", \"data\": {\"min\": 9.000000000000001e-08, \"max\": 1.1000000000000002e-07}}]}}, \"unit\": \"farad\"}}"
 			(at 0 0 0)
 			(layer "User.9")
@@
 			)
 		)
-		(property "Datasheet" "https://www.lcsc.com/datasheet/lcsc_datasheet_2206010216_UNI-ROYAL-Uniroyal-Elec-0402WGF1001TCE_C11702.pdf"
+		(property "Datasheet" ""
 			(at 0 0 0)
 			(layer "User.9")
@@
 			)
 		)
-		(property "Manufacturer" "UNI-ROYAL(Uniroyal Elec)"
+		(property "Manufacturer" "UNI-ROYAL"
 			(at 0 0 0)
 			(layer "User.9")
@@
 			)
 		)
-		(property "Datasheet" "https://www.lcsc.com/datasheet/lcsc_datasheet_2304140030_Samsung-Electro-Mechanics-CL05B104KO5NNNC_C1525.pdf"
+		(property "Datasheet" ""
 			(at 0 0 90)
 			(layer "User.9")
@@
 			)
 		)
-		(property "PARAM_capacitance" "{\"type\": \"Quantity_Interval_Disjoint\", \"data\": {\"intervals\": {\"type\": \"Numeric_Interval_Disjoint\", \"data\": {\"intervals\": [{\"type\": \"Numeric_Interval\", \"data\": {\"min\": 8.99999998509884e-08, \"max\": 1.1000000014901162e-07}}]}}, \"unit\": \"farad\"}}"
+		(property "PARAM_capacitance" "{\"type\": \"Quantity_Interval_Disjoint\", \"data\": {\"intervals\": {\"type\": \"Numeric_Interval_Disjoint\", \"data\": {\"intervals\": [{\"type\": \"Numeric_Interval\", \"data\": {\"min\": 9.000000000000001e-08, \"max\": 1.1000000000000002e-07}}]}}, \"unit\": \"farad\"}}"
 			(at 0 0 90)
 			(layer "User.9")
@@
 			)
 		)
-		(property "Datasheet" "https://www.lcsc.com/datasheet/lcsc_datasheet_2304140030_Samsung-Electro-Mechanics-CL10A475KO8NNNC_C19666.pdf"
+		(property "Datasheet" ""
 			(at 0 0 0)
 			(layer "User.9")
@@
 			)
 		)
-		(property "PARAM_capacitance" "{\"type\": \"Quantity_Interval_Disjoint\", \"data\": {\"intervals\": {\"type\": \"Numeric_Interval_Disjoint\", \"data\": {\"intervals\": [{\"type\": \"Numeric_Interval\", \"data\": {\"min\": 4.229999992996454e-06, \"max\": 5.170000007003546e-06}}]}}, \"unit\": \"farad\"}}"
+		(property "PARAM_capacitance" "{\"type\": \"Quantity_Interval_Disjoint\", \"data\": {\"intervals\": {\"type\": \"Numeric_Interval_Disjoint\", \"data\": {\"intervals\": [{\"type\": \"Numeric_Interval\", \"data\": {\"min\": 4.23e-06, \"max\": 5.1700000000000005e-06}}]}}, \"unit\": \"farad\"}}"
 			(at 0 0 0)
 			(layer "User.9")
@@
 			)
 		)
-		(property "Datasheet" "https://www.lcsc.com/datasheet/lcsc_datasheet_2206010045_UNI-ROYAL-Uniroyal-Elec-0402WGF5101TCE_C25905.pdf"
+		(property "Datasheet" ""
 			(at 0 0 0)
 			(layer "User.9")
@@
 			)
 		)
-		(property "Manufacturer" "UNI-ROYAL(Uniroyal Elec)"
+		(property "Manufacturer" "UNI-ROYAL"
 			(at 0 0 0)
 			(layer "User.9")
@@
 			)
 		)
-		(property "Datasheet" "https://www.lcsc.com/datasheet/lcsc_datasheet_2206010045_UNI-ROYAL-Uniroyal-Elec-0402WGF4701TCE_C25900.pdf"
+		(property "Datasheet" ""
 			(at 0 0 90)
 			(layer "User.9")
@@
 			)
 		)
-		(property "Manufacturer" "UNI-ROYAL(Uniroyal Elec)"
+		(property "Manufacturer" "UNI-ROYAL"
 			(at 0 0 90)
 			(layer "User.9")
